File: md/md.kicad_pcb (KiCad board)
At the start: 2 copper layers, 54.6 x 62.2 mm, 54 parts, among them J1 CONTROLL, J2 OUTA, J3 OUTB, J4 PWR_INPUT+, J5 PWR_INPUT-, J6 PWR_INPUT+, J7 PWR_INPUT+, J8 PWR_INPUT+, J9 PWR_INPUT+, Q1 IRFB7437PBF, Q2 IRFB7437PBF, Q3 IRFB7437PBF, Q4 IRFB7437PBF, U1 74HC00, U2 TLP2105, U3 IR7184S, U4 IR7184S, U5 LM7812_TO220

Commit message: fix capacitor arrangement
Parts:
- moved C7 4.58 mm to (17.8, 62.2), turned to 270 degrees
Routing:
- net +12V: track 141.1 -> 135.7 mm
- net GNDPWR: track 223.5 -> 226.7 mm, vias 2 -> 11
- net +24V: track 99.6 -> 97.2 mm
- added copper zone on B.Cu, net +24V
- removed copper zone on B.Cu, net +12V

Commit message: improve line design
Parts:
- turned D7 to 90 degrees
Routing:
- net +12V: track 135.7 -> 128.0 mm
- net +24V: track 97.2 -> 90.8 mm
Changed lines of the file:
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@@
     (thickness 1.6)
     (drawings 4)
-    (tracks 444)
+    (tracks 439)
     (zones 0)
     (modules 54)
@@
   )
   (module Diodes_SMD:D_SOD-123F (layer F.Cu)
-    (at 24.13 85.09 270)
+    (at 24.13 85.09 90)
     (descr D_SOD-123F)
     (tags D_SOD-123F)
     (attr smd)
-    (fp_text reference D7 (at -0.127 -1.905 270) (layer F.SilkS)
-      (effects (font (size 1 1) (thickness 0.15)))
-    )
-    (fp_text value SS2040FL (at 0 2.1 270) (layer F.Fab)
-      (effects (font (size 1 1) (thickness 0.15)))
-    )
-    (fp_text user %R (at -0.127 -1.905 270) (layer F.Fab)
+    (fp_text reference D7 (at -0.127 -1.905 90) (layer F.SilkS)
+      (effects (font (size 1 1) (thickness 0.15)))
+    )
+    (fp_text value SS2040FL (at 0 2.1 90) (layer F.Fab)
+      (effects (font (size 1 1) (thickness 0.15)))
+    )
+    (fp_text user %R (at -0.127 -1.905 90) (layer F.Fab)
       (effects (font (size 1 1) (thickness 0.15)))
     )
@@
     (fp_line (start -2.2 1) (end 1.65 1) (layer F.SilkS) (width 0.12))
     (fp_line (start -2.2 -1) (end 1.65 -1) (layer F.SilkS) (width 0.12))
-    (pad 1 smd rect (at -1.4 0 270) (size 1.1 1.1) (layers F.Cu F.Paste F.Mask)
-      (net 8 +24V))
-    (pad 2 smd rect (at 1.4 0 270) (size 1.1 1.1) (layers F.Cu F.Paste F.Mask)
+    (pad 1 smd rect (at -1.4 0 90) (size 1.1 1.1) (layers F.Cu F.Paste F.Mask)
+      (net 8 +24V))
+    (pad 2 smd rect (at 1.4 0 90) (size 1.1 1.1) (layers F.Cu F.Paste F.Mask)
       (net 4 +12V))
     (model ${KISYS3DMOD}/Diodes_SMD.3dshapes/D_SOD-123F.wrl
@@
   (segment (start 15.335 74.93) (end 17.875 72.39) (width 0.6) (layer F.Cu) (net 4))
   (segment (start 15.24 74.93) (end 15.335 74.93) (width 0.6) (layer F.Cu) (net 4))
-  (segment (start 26.489999 84.130001) (end 24.13 86.49) (width 0.6) (layer F.Cu) (net 4))
   (segment (start 53.037745 77.662249) (end 53.352745 77.347249) (width 0.25) (layer F.Cu) (net 4))
   (segment (start 53.037745 79.252249) (end 53.037745 77.662249) (width 0.25) (layer F.Cu) (net 4))
@@
   (segment (start 58.59 91.665002) (end 55.510001 94.745001) (width 0.6) (layer F.Cu) (net 4))
   (segment (start 28.070001 94.745001) (end 21.59 88.265) (width 0.6) (layer F.Cu) (net 4))
-  (segment (start 23.179998 82.55) (end 26.489999 82.55) (width 0.6) (layer F.Cu) (net 4))
-  (segment (start 21.59 84.139998) (end 23.179998 82.55) (width 0.6) (layer F.Cu) (net 4))
   (segment (start 21.59 88.265) (end 21.59 84.139998) (width 0.6) (layer F.Cu) (net 4))
-  (segment (start 26.489999 82.55) (end 26.489999 84.130001) (width 0.6) (layer F.Cu) (net 4))
   (segment (start 48.58 70.145) (end 48.58 71.12) (width 0.6) (layer F.Cu) (net 4))
   (segment (start 49.872001 68.852999) (end 48.58 70.145) (width 0.6) (layer F.Cu) (net 4))
@@
   (segment (start 15.24 77.789998) (end 21.59 84.139998) (width 0.6) (layer F.Cu) (net 4))
   (segment (start 15.24 74.93) (end 15.24 77.789998) (width 0.6) (layer F.Cu) (net 4))
+  (segment (start 22.039998 83.69) (end 24.13 83.69) (width 0.6) (layer F.Cu) (net 4))
+  (segment (start 21.59 84.139998) (end 22.039998 83.69) (width 0.6) (layer F.Cu) (net 4))
   (segment (start 34.29 58.59) (end 31.7 58.59) (width 0.25) (layer F.Cu) (net 5))
   (segment (start 25.4 64.89) (end 25.4 66.04) (width 0.25) (layer F.Cu) (net 5))
@@
   (segment (start 22.13 76.74) (end 20.32 74.93) (width 0.6) (layer F.Cu) (net 8))
   (segment (start 24.13 76.74) (end 22.13 76.74) (width 0.6) (layer F.Cu) (net 8))
-  (segment (start 23.029999 87.480001) (end 23.179998 87.63) (width 0.6) (layer F.Cu) (net 8))
-  (segment (start 24.13 83.69) (end 23.029999 84.790001) (width 0.6) (layer F.Cu) (net 8))
-  (segment (start 23.029999 84.790001) (end 23.029999 87.480001) (width 0.6) (layer F.Cu) (net 8))
-  (segment (start 25.080002 87.63) (end 28.255002 84.455) (width 0.6) (layer F.Cu) (net 8))
-  (segment (start 23.179998 87.63) (end 25.080002 87.63) (width 0.6) (layer F.Cu) (net 8))
-  (segment (start 28.255002 77.154998) (end 30.48 74.93) (width 0.6) (layer F.Cu) (net 8))
-  (segment (start 28.255002 84.455) (end 28.255002 77.154998) (width 0.6) (layer F.Cu) (net 8))
   (segment (start 24.13 69.755) (end 24.035 69.755) (width 0.6) (layer F.Cu) (net 8))
   (segment (start 20.930251 61.879749) (end 20.930251 53.950251) (width 1.8) (layer B.Cu) (net 8))
@@
   (segment (start 21.595 72.29) (end 24.13 69.755) (width 0.6) (layer F.Cu) (net 8))
   (segment (start 21.595 72.39) (end 21.595 72.29) (width 0.6) (layer F.Cu) (net 8))
+  (segment (start 24.13 86.49) (end 25.28 86.49) (width 0.6) (layer F.Cu) (net 8))
+  (segment (start 30.48 76.202792) (end 30.48 74.93) (width 0.6) (layer F.Cu) (net 8))
+  (segment (start 30.48 81.29) (end 30.48 76.202792) (width 0.6) (layer F.Cu) (net 8))
+  (segment (start 25.28 86.49) (end 30.48 81.29) (width 0.6) (layer F.Cu) (net 8))
   (segment (start 53.89338 68.154881) (end 54.71488 68.154881) (width 0.25) (layer F.Cu) (net 9))
   (segment (start 54.71488 68.154881) (end 54.918762 67.950999) (width 0.25) (layer F.Cu) (net 9))
@@
     (connect_pads (clearance 0.508))
     (min_thickness 0.254)
-    (fill yes (arc_segments 16) (thermal_gap 0.508) (thermal_bridge_width 0.508))
+    (fill (arc_segments 16) (thermal_gap 0.508) (thermal_bridge_width 0.508))
     (polygon
       (pts
@@
     (connect_pads (clearance 0.508))
     (min_thickness 0.254)
-    (fill yes (arc_segments 16) (thermal_gap 0.508) (thermal_bridge_width 0.508))
+    (fill (arc_segments 16) (thermal_gap 0.508) (thermal_bridge_width 0.508))
     (polygon
       (pts
@@
     (connect_pads yes (clearance 0.508))
     (min_thickness 0.254)
-    (fill yes (arc_segments 16) (thermal_gap 0.508) (thermal_bridge_width 0.508))
+    (fill (arc_segments 16) (thermal_gap 0.508) (thermal_bridge_width 0.508))
     (polygon
       (pts
@@
     (connect_pads yes (clearance 0.508))
     (min_thickness 0.254)
-    (fill yes (arc_segments 16) (thermal_gap 0.508) (thermal_bridge_width 0.508))
+    (fill (arc_segments 16) (thermal_gap 0.508) (thermal_bridge_width 0.508))
     (polygon
       (pts
@@
     (connect_pads yes (clearance 0.508))
     (min_thickness 0.254)
-    (fill yes (arc_segments 16) (thermal_gap 0.508) (thermal_bridge_width 0.508))
+    (fill (arc_segments 16) (thermal_gap 0.508) (thermal_bridge_width 0.508))
     (polygon
       (pts
@@
     (connect_pads yes (clearance 0.508))
     (min_thickness 0.254)
-    (fill yes (arc_segments 16) (thermal_gap 0.508) (thermal_bridge_width 0.508))
+    (fill (arc_segments 16) (thermal_gap 0.508) (thermal_bridge_width 0.508))
     (polygon
       (pts
@@
     (connect_pads (clearance 0.508))
     (min_thickness 0.254)
-    (fill yes (arc_segments 16) (thermal_gap 0.508) (thermal_bridge_width 0.508))
+    (fill (arc_segments 16) (thermal_gap 0.508) (thermal_bridge_width 0.508))
     (polygon
       (pts

Commit message: complete md
Parts:
- added REF**: MountingHole_3.2mm_M3, Mounting_Holes:MountingHole_3.2mm_M3, F.Cu at (8.26, 48.3)
- added REF**: MountingHole_3.2mm_M3, Mounting_Holes:MountingHole_3.2mm_M3, F.Cu at (63.5, 48.3)
- added REF**: MountingHole_3.2mm_M3, Mounting_Holes:MountingHole_3.2mm_M3, F.Cu at (62.2, 92.1)
- added REF**: MountingHole_3.2mm_M3, Mounting_Holes:MountingHole_3.2mm_M3, F.Cu at (8.26, 92.1)
- moved J4 18.0 mm to (8.26, 66.0)
- moved J5 16.9 mm to (8.26, 71.1)
- moved C1 7.24 mm to (59.7, 76.8), turned to 180 degrees
- moved C13 7.10 mm to (14.6, 65.4)
- moved JP1 7.01 mm to (20.3, 65.4)
- moved C7 6.40 mm to (16.5, 56.0)
- moved J1 5.24 mm to (58.4, 62.2)
- moved C12 5.08 mm to (19.1, 71.8), turned to 180 degrees
- moved D7 4.45 mm to (24.1, 80.6), turned to 270 degrees
- moved C6 4.44 mm to (24.1, 74.3)
- moved D10 2.24 mm to (63.6, 81.9)
- moved D11 2.24 mm to (63.6, 79.4)
- moved U1 2.01 mm to (61.6, 70.5)
- moved R11 1.92 mm to (59.4, 81.9)
- moved R12 1.92 mm to (59.4, 79.4)
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Connections:
- C2 pad 1: GND -> GNDPWR
Routing:
- net GND: track 58.7 -> 37.2 mm
- net +12V: track 128.0 -> 147.3 mm
- net +24V: track 90.8 -> 104.4 mm
- net Net-(Q1-Pad1): track 38.6 -> 26.8 mm
- net Net-(Q4-Pad1): track 33.5 -> 23.0 mm, vias 2 -> 1
- net +5V: track 35.8 -> 26.8 mm, vias 4 -> 1
- net /PWM: track 31.7 -> 26.4 mm, vias 1 -> 2
- net Net-(C5-Pad2): track 57.6 -> 60.8 mm, vias 2 -> 0
- net /OUTB: track 18.4 -> 16.3 mm
- net /DIR: track 42.2 -> 40.7 mm, vias 4 -> 2
- net Net-(R8-Pad2): track 9.87 -> 8.77 mm
- net Net-(R14-Pad1): track 2.95 -> 2.00 mm
- net Net-(D9-Pad2): track 2.88 -> 1.95 mm
- net Net-(D8-Pad2): track 2.88 -> 1.95 mm
- net Net-(D11-Pad2): track 2.88 -> 1.95 mm
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Other:
- board size 54.6 x 62.2 mm -> 62.2 x 62.2 mm
